File: msp_dj_chip/_autosave-msp_dj_chip.kicad_sch (KiCad schematic)
At the start: 7 parts, among them U1 DAC60502

Commit message: Add files via upload
Parts:
- removed U1: DAC60502, symbol bernie_symbols:DAC
- removed U2: ~, symbol Project_Symbols:MCU_MSPM0G3507
- added C1, C2: 100nF, Capacitor_SMD:C_0402_1005Metric, symbol Device:C_Small
- added C10, C12, C8, C9: 100n, Capacitor_SMD:C_0402_1005Metric, symbol Device:C_Small
- added C11: 4u7, symbol Device:C_Polarized_Small
- added C13: u1F, symbol Device:C_Small
- added C14: 10uF, symbol Device:C_Small
- added C15: u47, symbol Device:C_Small
- added C16: 10nF, symbol Device:C_Small
- added C17, C18: 15pF, symbol Device:C_Small
- added C3: 150nF, Capacitor_SMD:C_0402_1005Metric, symbol Device:C_Small
- added C4, C5: 10u, Capacitor_SMD:C_0603_1608Metric, symbol Device:C_Small
- added C6, C7: 47p, Capacitor_SMD:C_0402_1005Metric, symbol Device:C_Small
- added D1, D2, D3, D4, D5: LED_Small_Filled, LED_SMD:LED_0603_1608Metric, symbol Device:LED_Small_Filled
- added FB1: 600R@100Mhz, symbol Device:FerriteBead_Small
- added J1, J2: Conn_01x04_Pin, symbol Connector:Conn_01x04_Pin
- added J10, J11, J12, J13, J14, J15, J16, J17, J18, J19, J20, J21, J3, J4, J5, J6, J9: Conn_01x02_Socket, symbol Connector:Conn_01x02_Socket
- added J22, J23: Conn_01x06_Socket, symbol Connector:Conn_01x06_Socket
- added J8: Conn_02x05_Odd_Even, symbol Connector_Generic:Conn_02x05_Odd_Even
- added R10, R11, R18, R29, R30: 2K2, symbol Device:R_Small
- added R12, R13: 27R, symbol Device:R_Small
- added R14, R15, R16: 10K, symbol Device:R_Small
- added R17: 330R, symbol Device:R_Small
- added R19, R20: 5K1, symbol Device:R_Small
- added R21, R22: 0R, symbol Device:R_Small
- added R23, R25, R26: 47K, symbol Device:R_Small
- added R24: 100K, symbol Device:R_Small
- added R27, R28: 1R, symbol Device:R_Small
- added R33, R6, R8, R9: 1K, symbol Device:R_Small
- added R7: 10k, symbol Device:R_Small
- added TP1: TestPoint, symbol Connector:TestPoint
- added U1: ~, symbol Project_Symbols:RS485_THVD2412
- added U2: DAC60502, symbol Project_Symbols:DAC_60502
- added U3: ~, symbol Project_Symbols:OpAmp_NCV272
- added U4: NCP1117-3.3_SOT223, Package_TO_SOT_SMD:SOT-223-3_TabPin2, symbol Regulator_Linear:NCP1117-3.3_SOT223
- added U5: ~, symbol Project_Symbols:ftdi_FT231X
- added U6: ~, symbol Project_Symbols:MCU_MSPM0G3507
- added U8: NCV272DMR2G, symbol Project_Symbols:OpAmp_NCV272
- added Y1: Crystal_GND24_Small, symbol Device:Crystal_GND24_Small
- R1: value 1K -> 4K7; footprint Resistor_SMD:R_0603_1608Metric -> (none); now not fitted
- R2: footprint Resistor_SMD:R_0603_1608Metric -> (none)
- R3: footprint Resistor_SMD:R_0603_1608Metric -> (none); now not fitted
- R4, R5: value 1K -> 120R; footprint Resistor_SMD:R_0603_1608Metric -> (none)
Connections:
- net +3V3: now also J1.3 (Pin_3), R17.1; no longer R1.1, R2.1, R3.1, R4.1, R5.1
- net GND: now also C1.2, C10.2, C11.2, C12.2, C13.2, C14.2, C15.2, C16.2, C17.1, C18.1, C2.2, C3.2, C4.2, C5.2, C6.2, C7.2, C8.2, C9.2, D4.1 (K), D5.1 (K), J1.2 (Pin_2), J1.4 (Pin_4), J22.1 (Pin_1), J23.1 (Pin_1), J23.2 (Pin_2), J8.3 (Pin_3), J8.5 (Pin_5), J8.7 (Pin_7), J8.9 (Pin_9), R15.2, R16.2, R19.1, R20.2, R24.1, R27.1, R28.1, R6.2, R8.1, R9.1, U1.11 (PAD), U1.5 (GND), U3.4 (VSS), U4.1 (GND), U5.16 (GND), U5.6 (GND), U8.4 (VSS); no longer R1.2, R2.2, R4.2, R5.2
- net NSYNC: now also R7.2, U2.7 (NSYNC)
- net RSTSEL: now also U2.3 (RSTSEL)
- net SCLK: now also U2.6 (SCLK)
- net SDIN: now also U2.8 (SDIN)
- net SPI: now also R6.1, U2.5 (SPI)
- new net: D2.2 (A), R16.1
- new net: J8.10 (Pin_10), R22.1
- new net: C3.1, U2.10 (VREFIO)
- new net: C11.1, C12.1, D3.1 (K), FB1.1
- new net: J8.1 (Pin_1), R21.2
- new net: R29.1, R33.2, U8.2 (IN-1)
- new net: R30.1, U8.3 (IN+1)
- new net: D5.2 (A), R18.2
- new net: R10.1, R8.2, U3.2 (IN-1)
- new net: R11.1, R9.2, U3.6 (IN-2)
- new net: D2.1 (K), U5.10 (CBUS2)
- new net: R12.2, U5.11 (USBDP)
- new net: R13.2, U5.12 (USBDM)
- new net: D1.1 (K), U5.17 (CBUS1)
- new net: D4.2 (A), R17.2
- new net: C6.1, R13.1
- new net: D1.2 (A), R15.1
- new net: C16.1, R23.1, U6.38 (NRST)
- new net: C15.1, U6.32 (VCORE)
- new net: C7.1, R12.1
- new net +24V: J1.1 (Pin_1), J10.2 (Pin_2), J11.2 (Pin_2), J12.2 (Pin_2), J13.2 (Pin_2), J14.2 (Pin_2), J15.2 (Pin_2), J16.2 (Pin_2), J17.2 (Pin_2), J18.2 (Pin_2), J19.2 (Pin_2), J20.2 (Pin_2), J21.2 (Pin_2), J3.2 (Pin_2), J4.2 (Pin_2), J5.2 (Pin_2), J6.2 (Pin_2), R18.1, R28.2, U3.8 (VDD), U6.9 (PA16), U8.8 (VDD)
- new net +3.3V: C1.1, C13.1, C14.1, C2.1, C5.1, C8.1, R1.1, R14.1, R2.1, R21.1, R23.2, R25.2, R26.2, R7.1, U1.10 (V_{CC}), U2.1 (VDD), U4.2 (VO), U5.3 (VCCIO), U6.40 (VDD)
- new net ANALOG_IN0: J2.2 (Pin_2)
- new net ANALOG_IN1: J2.1 (Pin_1)
- new net CC1: J22.5 (Pin_5), R19.2
- new net CC2: J22.4 (Pin_4), R20.1
- new net D: U1.4 (D)
- new net DAC OUT0: R10.2, R29.2, R30.2, U3.1 (OUT_1), U8.1 (OUT_1)
- new net DAC OUT1: R11.2, U3.7 (OUT_2)
- new net DAC_0: R33.1, U6.54 (PA8)
- new net DAC_OUT0: J2.4 (Pin_4)
- new net DAC_OUT1: J2.3 (Pin_3)
- new net DE: R3.1, U1.3 (DE)
- new net FTDI 3V3: TP1.1, U5.13 (3V3OUT)
- new net FTDI_RX: U6.11 (PA18)
- new net FTDI_TX: U6.10 (PA17)
- new net HFXIN: C17.2, U6.24 (PA23), Y1.1
- new net HFXOUT: C18.2, U6.25 (PA24), Y1.3
- new net OUT_0: J3.1 (Pin_1)
- new net OUT_1: J4.1 (Pin_1)
- new net OUT_10: J15.1 (Pin_1)
- new net OUT_11: J16.1 (Pin_1)
- new net OUT_12: J17.1 (Pin_1)
- new net OUT_13: J18.1 (Pin_1), J19.1 (Pin_1)
- new net OUT_14: J20.1 (Pin_1)
- new net OUT_15: J21.1 (Pin_1)
- new net OUT_2: J5.1 (Pin_1)
- new net OUT_3: J6.1 (Pin_1)
- new net OUT_4: J9.1 (Pin_1)
- new net OUT_5: J10.1 (Pin_1)
- new net OUT_6: J11.1 (Pin_1)
- new net OUT_7: J12.1 (Pin_1)
- new net OUT_8: J13.1 (Pin_1)
- new net OUT_9: J14.1 (Pin_1)
- new net R: R2.2, U1.1 (R)
- new net RE: R1.2, U1.2 (RE)
- new net RS485_RX: R26.1, U6.34 (PA1)
- new net RS485_TX: R25.1, U6.33 (PA_0/FCC_IN)
- new net RX+: J23.3 (Pin_3), R5.1, U1.9 (A)
- new net RX-: J23.4 (Pin_4), R5.2, U1.8 (B)
- new net SOL_OUT_0: U6.1 (PB13)
- new net SOL_OUT_1: U6.2 (PB14)
- new net SOL_OUT_10: U6.18 (PA22)
- new net SOL_OUT_11: U6.19 (PB20)
- new net SOL_OUT_12: U6.20 (PB21)
- new net SOL_OUT_13: U6.21 (PB22)
- new net SOL_OUT_14: U6.22 (PB23)
- new net SOL_OUT_15: U6.23 (PB24)
- new net SOL_OUT_2: U6.3 (PB15)
- new net SOL_OUT_3: U6.4 (PB16)
- new net SOL_OUT_4: U6.5 (PA12/FCC_IN)
- new net SOL_OUT_5: U6.6 (PA13)
- new net SOL_OUT_6: U6.14 (PB17)
- new net SOL_OUT_7: U6.15 (PB18)
- new net SOL_OUT_8: U6.16 (PB19)
- new net SOL_OUT_9: U6.17 (PA21)
- new net SPI_0_CS: R24.2, U6.42 (PA2)
- new net SPI_PICO: U6.7 (PA14/A0_12/CLK_OUT)
- new net SPI_POCI: U6.56 (PA10)
- new net SPI_SCLK: U6.57 (PA11)
- new net SWCLK: U6.13 (PA20)
- new net SWDIO: U6.12 (PA19)
- new net TX+: J23.5 (Pin_5), R4.1, U1.6 (Y)
- new net TX-: J23.6 (Pin_6), R4.2, U1.7 (Z)
- new net UART2 RX: U5.20 (TXD)
- new net UART2 TX: U5.4 (RXD)
- new net USB_D+: J22.2 (Pin_2)
- new net USB_D-: J22.3 (Pin_3)
- new net VBUS: C4.1, D3.2 (A), J22.6 (Pin_6), R27.2, U4.3 (VI), U6.8 (PA15/A1_0)
- new net VBUS_FILT: C10.1, C9.1, FB1.2, U5.15 (VCC)
- new net VOUTA: U2.2 (VOUTA), U3.3 (IN+1)
- new net VOUTB: U2.9 (VOUTB), U3.5 (IN+2)
- new net nRESET: R22.2, U5.14 (~{RESET})
- no-connect marks 0 -> 13
Other:
- note added: "24 Current Sense"
- note added: "ANALOGUE OUT"
- note added: "DAC"
- note added: "FTDI"
- note added: "LDO"
- note added: "OP-AMP"
- note added: "POWER + INPUT"
- note added: "PROGRAMMING HEADER"
- note added: "RS485"
- note added: "RS485 OUTPUT"
- note added: "SOL OUT"
- note added: "USB"
- note added: "VBUS Current Sense"

Commit message: updated changes
Connections:
- net DAC_0: now also U6.8 (PA15/A1_0); no longer U6.54 (PA8)
- net VBUS: no longer U6.8 (PA15/A1_0)
Other:
- added sheet led-driver (led_driver.kicad_sch)
- added sheet solenoid-driver-boards-dj (solenoid-driver-boards-dj.kicad_sch)
- moved on the sheet: R29, R30, R33, U8A, U8B
