File: msp_dj_chip/solenoid-driver-boards-dj.kicad_sch (KiCad schematic)
At the start: 208 parts, among them Q1 PMGD780SN, Q2 PMGD780SN, Q3 PMGD780SN, Q4 PMGD780SN, Q5 PMGD780SN, Q6 PMGD780SN, Q7 PMGD780SN, Q8 PMGD780SN, U16 NCV272DMR2G, U17 NCV272DMR2G, U18 NCV272DMR2G, U19 NCV272DMR2G, U20 NCV272DMR2G, U21 NCV272DMR2G, U22 NCV272DMR2G, U23 NCV272DMR2G

Commit message: some changes
Connections:
- net GPIO_INPUT_04: now reaches R72.1
- net GPIO_INPUT_10: now reaches R96.1
- net OUT_04: now reaches Q3.6 (D1), TP28.1
- net OUT_02: now reaches Q1.6 (D1), TP18.1
- net OUT_14: now reaches Q8.6 (D1), TP78.1
- net OUT_15: now reaches Q8.3 (D2), TP80.1
- net OUT_09: now reaches Q6.3 (D2), TP60.1
- net GPIO_INPUT_00: now reaches R48.1
- net OUT_06: now reaches Q4.6 (D1), TP38.1
- net OUT_10: now reaches Q5.6 (D1), TP54.1
- net OUT_08: now reaches Q6.6 (D1), TP58.1
- net OUT_05: now reaches Q3.3 (D2), TP30.1
- net OUT_01: now reaches Q2.3 (D2), TP10.1
- net OUT_12: now reaches Q7.6 (D1), TP74.1
- net GPIO_INPUT_08: now reaches R100.1
- net GPIO_INPUT_12: now reaches R120.1
- net OUT_07: now reaches Q4.3 (D2), TP40.1
- net OUT_00: now reaches Q2.6 (D1), TP6.1
- net GPIO_INPUT_15: now reaches R126.1
- net OUT_11: now reaches Q5.3 (D2), TP56.1
- net GPIO_INPUT_13: now reaches R122.1
- net GPIO_INPUT_03: now reaches R62.1
- net GPIO_INPUT_06: now reaches R84.1
- net GPIO_INPUT_09: now reaches R102.1
- net OUT_13: now reaches Q7.3 (D2), TP76.1
- net GPIO_INPUT_01: now reaches R54.1
- net OUT_03: now reaches Q1.3 (D2), TP20.1
- net GPIO_INPUT_05: now reaches R74.1
- net GPIO_INPUT_14: now reaches R124.1
- net GPIO_INPUT_02: now reaches R60.1
- net GPIO_INPUT_11: now reaches R98.1
- net GPIO_INPUT_07: now reaches R86.1

Commit message: Update TODO list
Connections:
- net SENSE_00: now reaches Q2.1 (S1), R50.2, R52.2, TP4.1
Other:
- note added: "Put SENSE pins like that for all SOL OUTs"
- moved on the sheet: TP4
Changed lines of the file:
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@@
 		)
 	)
+	(text "Put SENSE pins like that for all SOL OUTs"
+		(exclude_from_sim no)
+		(at 113.538 58.674 0)
+		(effects
+			(font
+				(size 1.27 1.27)
+			)
+		)
+	)
 	(text "SOL_OUT_10-11"
 		(exclude_from_sim no)
@@
 	)
 	(junction
+		(at 91.44 62.23)
+		(diameter 0)
+		(color 0 0 0 0)
+	)
+	(junction
 		(at 269.24 177.8)
 		(diameter 0)
@@
 	(wire
 		(pts
+			(xy 88.9 62.23) (xy 91.44 62.23)
+		)
+		(stroke
+			(width 0)
+			(type default)
+		)
+	)
+	(wire
+		(pts
 			(xy 62.23 93.98) (xy 68.58 93.98)
 		)
@@
 	(wire
 		(pts
-			(xy 88.9 34.29) (xy 88.9 39.37)
+			(xy 88.9 36.83) (xy 88.9 39.37)
 		)
 		(stroke
@@
 	(wire
 		(pts
+			(xy 91.44 62.23) (xy 93.98 62.23)
+		)
+		(stroke
+			(width 0)
+			(type default)
+		)
+	)
+	(wire
+		(pts
 			(xy 130.81 64.77) (xy 135.89 64.77)
 		)
@@
 	)
 	(hierarchical_label "OUT_00"
-		(shape input)
-		(at 88.9 34.29 0)
+		(shape output)
+		(at 88.9 36.83 90)
 		(effects
 			(font
@@
 		)
 	)
+	(hierarchical_label "SENSE_00"
+		(shape output)
+		(at 93.98 62.23 0)
+		(effects
+			(font
+				(size 1.27 1.27)
+			)
+			(justify left)
+		)
+	)
 	(hierarchical_label "GPIO_INPUT_01"
 		(shape input)
@@
 	(symbol
 		(lib_id "Connector:TestPoint")
-		(at 88.9 62.23 270)
+		(at 91.44 62.23 0)
 		(unit 1)
 		(exclude_from_sim no)
@@
 		(dnp no)
 		(property "Reference" "TP4"
-			(at 93.98 61.976 90)
+			(at 91.186 57.15 90)
 			(effects
 				(font
@@
 		)
 		(property "Value" "TestPoint"
-			(at 93.98 63.4999 90)
+			(at 92.7099 57.15 90)
 			(effects
 				(font
@@
 		)
 		(property "Footprint" ""
-			(at 88.9 67.31 0)
+			(at 96.52 62.23 0)
 			(effects
 				(font
@@
 		)
 		(property "Datasheet" "~"
-			(at 88.9 67.31 0)
+			(at 96.52 62.23 0)
 			(effects
 				(font
@@
 		)
 		(property "Description" "test point"
-			(at 88.9 62.23 0)
+			(at 91.44 62.23 0)
 			(effects
 				(font
