File: msp_dj_chip/solenoid-driver-boards-dj.kicad_sch (KiCad schematic)
At the start: 208 parts, among them Q1 PMGD780SN, Q2 PMGD780SN, Q3 PMGD780SN, Q4 PMGD780SN, Q5 PMGD780SN, Q6 PMGD780SN, Q7 PMGD780SN, Q8 PMGD780SN, U16 NCV272DMR2G, U17 NCV272DMR2G, U18 NCV272DMR2G, U19 NCV272DMR2G, U20 NCV272DMR2G, U21 NCV272DMR2G, U22 NCV272DMR2G, U23 NCV272DMR2G

Commit message: labeling ERC checking
Parts:
- removed TP61: TestPoint, symbol Connector:TestPoint
- added TP59, TP78: TestPoint, symbol Connector:TestPoint
- renumbered C29 to C27, C30 to C28, C27 to C29, C28 to C30, Q2 to Q1, Q1 to Q2, Q6 to Q5, Q5 to Q6, R116 to R100, R117 to R101, R120 to R102, R121 to R103, R122 to R104, R123 to R105, R124 to R106, R125 to R107, R126 to R108, R127 to R109, R128 to R110, R129 to R111, R130 to R112, R131 to R113, R132 to R114, R133 to R115, R134 to R116, R135 to R117, R136 to R118, R137 to R119, R138 to R120, R139 to R121, R140 to R122, R141 to R123, R142 to R124, R143 to R125, R48 to R30, R49 to R31, R54 to R32, R55 to R33, R60 to R34, R61 to R35, R62 to R36, R63 to R37, R50 to R38, R56 to R39, R64 to R40, R65 to R41, R53 to R42, R57 to R43, R66 to R44, R67 to R45, R51 to R46, R58 to R47, R68 to R48, R69 to R49, R52 to R50, R59 to R51, R70 to R52, R71 to R53, R72 to R54, R73 to R55, R74 to R56, R75 to R57, R84 to R58, R85 to R59, R86 to R60, R87 to R61, R76 to R62, R77 to R63, R78 to R64, R79 to R65, R88 to R66, R89 to R67, R90 to R68, R91 to R69, R80 to R70, R81 to R71, R92 to R72, R93 to R73, R82 to R74, R83 to R75, R94 to R76, R95 to R77, R100 to R78, R101 to R79, R102 to R80, R103 to R81, R96 to R82, R97 to R83, R98 to R84, R99 to R85, R106 to R86, R107 to R87, R110 to R88, R111 to R89, R104 to R90, R105 to R91, R108 to R92, R109 to R93, R114 to R94, R115 to R95, R112 to R96, R113 to R97, R118 to R98, R119 to R99, TP5 to TP10, TP9 to TP11, TP16 to TP12, TP17 to TP13, TP6 to TP14, TP10 to TP15, TP18 to TP16, TP20 to TP17, TP4 to TP18, TP11 to TP19, TP19 to TP20, TP32 to TP24, TP33 to TP25, TP24 to TP26, TP25 to TP27, TP34 to TP28, TP35 to TP29, TP7 to TP3, TP26 to TP30, TP27 to TP31, TP36 to TP32, TP37 to TP33, TP28 to TP34, TP30 to TP35, TP38 to TP36, TP40 to TP37, TP29 to TP38, TP31 to TP39, TP12 to TP4, TP39 to TP40, TP44 to TP42, TP45 to TP43, TP42 to TP44, TP43 to TP45, TP48 to TP46, TP49 to TP47, TP46 to TP48, TP47 to TP49, TP13 to TP5, TP52 to TP50, TP53 to TP51, TP50 to TP52, TP51 to TP53, TP58 to TP54, TP60 to TP55, TP54 to TP56, TP56 to TP57, TP59 to TP58, TP3 to TP6, TP55 to TP60, TP57 to TP61, TP8 to TP7, TP76 to TP75, TP78 to TP76, TP80 to TP77, TP75 to TP79, TP14 to TP8, TP77 to TP80, TP79 to TP81, TP81 to TP82, TP15 to TP9, U17 to U10, U18 to U11, U19 to U12, U21 to U13, U20 to U14, U22 to U15, U23 to U16, U16 to U9
Connections:
- net SENSE_07: now reaches Q4.4 (S2), R67.2, R77.2, TP41.1
- net SENSE_13: now reaches Q7.4 (S2), R111.2, R123.2, TP80.1
- net SENSE_14: now reaches Q8.1 (S1), R114.2, R124.2, TP81.1
- net SENSE_04: now reaches Q3.1 (S1), R62.2, R74.2, TP38.1
- net SENSE_15: now reaches Q8.4 (S2), R115.2, R125.2, TP82.1
- net SENSE_06: now reaches Q4.1 (S1), R66.2, R76.2, TP40.1
- net SENSE_05: now reaches Q3.4 (S2), R63.2, R75.2, TP39.1
- net SENSE_03: now reaches Q2.4 (S2), R41.2, R53.2, TP21.1
- net SENSE_12: now reaches Q7.1 (S1), R110.2, R122.2, TP79.1
- net SENSE_12: now also TP78.1
- net SENSE_02: now reaches Q2.1 (S1), R40.2, R52.2, TP20.1
- net SENSE_10: now reaches Q6.1 (S1), R100.2, R90.2, TP60.1
- net SENSE_01: now reaches Q1.4 (S2), R39.2, R51.2, TP19.1
- net SENSE_08: now reaches Q5.1 (S1), R86.2, R98.2, TP58.1
- net SENSE_11: now reaches Q6.4 (S2), R101.2, R91.2, TP61.1
- net SENSE_09: now reaches Q5.4 (S2), R87.2, R99.2
- net SENSE_09: now also TP59.1
Other:
- moved on the sheet: R77, TP19, TP20, TP21, TP38, TP39, TP40, TP41, TP58, TP60, TP61, TP79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

Commit message: updating footprint assignments
Parts:
- C19, C20, C21, C22, C23, C24, C25, C26, C27, C28, C29, C30, C31, C32, C33, C34: footprint (none) -> Capacitor_SMD:C_0603_1608Metric
- R100, R101, R102, R103, R104, R105, R106, R107, R108, R109, R110, R111, R112, R113, R114, R115, R116, R117, R118, R119, R120, R121, R122, R123, R124, R125, R30, R31, R32, R33, R34, R35, R36, R37, R38, R39, R40, R41, R42, R43, R44, R45, R46, R47, R48, R49, R50, R51, R52, R53, R54, R55, R56, R57, R58, R59, R60, R61, R62, R63, R64, R65, R66, R67, R68, R69, R70, R71, R72, R73, R74, R75, R76, R77, R78, R79, R80, R81, R82, R83, R84, R85, R86, R87, R88, R89, R90, R91, R92, R93, R94, R95, R96, R97, R98, R99: footprint (none) -> Resistor_SMD:R_0603_1608Metric
- TP10, TP11, TP12, TP13, TP14, TP15, TP16, TP17, TP18, TP19, TP2, TP20, TP21, TP22, TP23, TP24, TP25, TP26, TP27, TP28, TP29, TP3, TP30, TP31, TP32, TP33, TP34, TP35, TP36, TP37, TP38, TP39, TP4, TP40, TP41, TP42, TP43, TP44, TP45, TP46, TP47, TP48, TP49, TP5, TP50, TP51, TP52, TP53, TP54, TP55, TP56, TP57, TP58, TP59, TP6, TP60, TP61, TP62, TP63, TP64, TP65, TP66, TP67, TP68, TP69, TP7, TP70, TP71, TP72, TP73, TP74, TP75, TP76, TP77, TP78, TP79, TP8, TP80, TP81, TP82, TP9: footprint (none) -> TestPoint:TestPoint_Pad_2.0x2.0mm
