File: msp_dj_chip/msp_dj_chip.kicad_sch (KiCad schematic)
At the start: 110 parts, among them J1 Conn_01x04_Pin, J10 Conn_01x02_Socket, J11 Conn_01x02_Socket, J12 Conn_01x02_Socket, J13 Conn_01x02_Socket, J14 Conn_01x02_Socket, J15 Conn_01x02_Socket, J16 Conn_01x02_Socket, J17 Conn_01x02_Socket, J18 Conn_01x02_Socket, J19 Conn_01x02_Socket, J2 Conn_01x06_Socket, J20 Conn_01x02_Socket, J21 Conn_02x05_Odd_Even, J22 Conn_01x04_Pin, J3 Conn_01x06_Socket, J4 Conn_01x02_Socket, J5 Conn_01x02_Socket, J6 Conn_01x02_Socket, J7 Conn_01x02_Socket, J8 Conn_01x02_Socket, J9 Conn_01x02_Socket, SW1 SW_MEC_5E, U1 SSM6N7002KFU, U2 FT231XS-R, U3 THVD2442, U4 NCP1117-3.3_SOT223, U5 SSM6N7002KFU, U6 DAC60502, U7 NCV272DMR2G, U8 NCV272DMR2G, Y1 24 MHz

Commit message: Made all sheet to sheet global labels
Connections:
- net DAC_00 renamed DAC_0
Other:
- moved on the sheet: C18
